Commit message: Add Collision Tags

File: src/my_robot_description/urdf/arm.xacro (robot description, xacro)
@@ -9,4 +9,10 @@
             <material name="grey" />
         </visual>
+        <collision>
+            <geometry>
+                <box size="0.4 0.4 0.1" />
+            </geometry>
+            <origin xyz="0 0 0.05" rpy="0 0 0" />
+        </collision>
     </link>
     <link name="shoulder_link">
@@ -18,4 +24,10 @@
             <material name="blue" />
         </visual>
+        <collision>
+            <geometry>
+                <cylinder length="0.5" radius="0.1" />
+            </geometry>
+            <origin xyz="0 0 0.25" rpy="0 0 0" />
+        </collision>
     </link>
     <link name="arm_link">
@@ -27,4 +39,10 @@
             <material name="grey" />
         </visual>
+        <collision>
+            <geometry>
+                <cylinder length="0.6" radius="0.05" />
+            </geometry>
+            <origin xyz="0 0 0.3" rpy="0 0 0" />
+        </collision>
     </link>
     <link name="elbow_link">
@@ -36,4 +54,10 @@
             <material name="blue" />
         </visual>
+        <collision>
+            <geometry>
+                <cylinder length="0.1" radius="0.05" />
+            </geometry>
+            <origin xyz="0 0 0.05" rpy="0 0 0" />
+        </collision>
     </link>
     <link name="forearm_link">
@@ -45,4 +69,10 @@
             <material name="grey" />
         </visual>
+        <collision>
+            <geometry>
+                <cylinder length="0.5" radius="0.05" />
+            </geometry>
+            <origin xyz="0 0 0.25" rpy="0 0 0" />
+        </collision>
     </link>
     <link name="wrist_link">
@@ -54,4 +84,10 @@
             <material name="blue" />
         </visual>
+        <collision>
+            <geometry>
+                <box size="0.1 0.1 0.05" />
+            </geometry>
+            <origin xyz="0 0 0.025" rpy="0 0 0" />
+        </collision>
     </link>
     <link name="hand_link">
@@ -63,4 +99,10 @@
             <material name="grey" />
         </visual>
+        <collision>
+            <geometry>
+                <box size="0.1 0.1 0.02" />
+            </geometry>
+            <origin xyz="0 0 0.01" rpy="0 0 0" />
+        </collision>
     </link>
     <link name="tool_link" />

Commit message: Fix: Add Collision Tags

File: src/my_robot_description/urdf/arm.xacro (robot description, xacro)
@@ -26,5 +26,5 @@
         <collision>
             <geometry>
-                <cylinder length="0.5" radius="0.1" />
+                <box size="0.2 0.2 0.5"/>
             </geometry>
             <origin xyz="0 0 0.25" rpy="0 0 0" />
@@ -41,5 +41,5 @@
         <collision>
             <geometry>
-                <cylinder length="0.6" radius="0.05" />
+                <box size="0.1 0.1 0.6" />
             </geometry>
             <origin xyz="0 0 0.3" rpy="0 0 0" />
@@ -56,5 +56,5 @@
         <collision>
             <geometry>
-                <cylinder length="0.1" radius="0.05" />
+                <box size="0.1 0.1 0.1" />
             </geometry>
             <origin xyz="0 0 0.05" rpy="0 0 0" />
@@ -71,5 +71,5 @@
         <collision>
             <geometry>
-                <cylinder length="0.5" radius="0.05" />
+                <box size="0.1 0.1 0.5" />
             </geometry>
             <origin xyz="0 0 0.25" rpy="0 0 0" />
